File: ponderada_sem6_kicad/ponderada_sem6_kicad.kicad_pcb (KiCad board)
At the start: 2 copper layers, 6 parts, among them Q1 BC548, U1 Pico

Commit message: atualização de arquivos
Other:
- board outline added: 64 x 61.5 mm
Changed lines of the file:
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@@
 		)
+	)
+	(gr_rect
+		(start 95 79.5)
+		(end 159 141)
+		(stroke
+			(width 0.05)
+			(type default)
+		)
+		(fill none)
+		(layer "Edge.Cuts")
 	)
 	(segment
